File: project files/stlink/stlink.sch (KiCad schematic (older format))
At the start: 38 parts

Commit message: updates + references
Parts:
- added C?: 100nF, symbol Device:C
- added R? (x2): 220R, symbol Device:R
- added R? (x2): 47R, symbol Device:R
- added R?: 680R, symbol Device:R
- added R?: 10K, symbol Device:R
- R? (x3): value 100 -> 100R
- R? (x2): value 330 -> 330R
Connections:
- net +3V3: now also R?.2
- net AIN: now also C?.1
- net GNDREF: now also C?.2, R?.2
- net T_NRST_SWD: now also U?.18 (PB0)
- net T_NRST_SWIM: now also U?.42 (PB6), R?.1, R?.2, R?.2
- net T_SWIM: now also U?.22 (PB11), U?.45 (PB8), R?.1, R?.1, R?.2, R?.2
- net T_SWIM_IN: now reaches U?.21 (PB10)
- net T_SWIM_IN: now also U?.41 (PB5), U?.43 (PB7), U?.46 (PB9), R?.1
- net PC14: now reaches U?.3 (PC14)
- net PC14: now also R?.1
- new net T_NRST_SWIM_IN: R?.1
- no-connect marks 11 -> 10
Other:
- note added: "Don't solder this one!"
- note added: "Microcontroller core"
- note added: "Original boards use as ST-link V2.1:\n- STM32F103CBT6 : Nucleo 32 boards [STM8 and STM32F]\n- STM32F103CBT6TR : Nucleo 64 boards with STM8\nOriginal boards use as ST-Link V2:\n- STM32F103C8T6 : F4Discovery\n\nClones use STM32F101****"
- moved on the sheet: C?, R?, U?

Commit message: Added STDC14
Parts:
- added C?: 20pF, symbol Device:C
- added D?: BAT60A, Diode_SMD:D_SOD-323, symbol Diode:BAT60A
- added J?: STDC14, symbol Connector_Generic:Conn_02x07_Odd_Even
- added R?: 4K7, symbol Device:R
- added R?: 100R, symbol Device:R
Connections:
- net AIN: now also R?.1
- net GNDREF: now also C?.2, J?.11 (Pin_11), J?.5 (Pin_5), J?.7 (Pin_7), R?.2; no longer R?.1
- net T_NRST_SWD: no longer R?.1
- net T_NRST_SWIM: no longer R?.2
- net T_SWDCLK: no longer R?.1
- net T_SWDIO: no longer R?.1
- net T_SWIM: no longer R?.2
- net Self_NRST renamed Self_NRSTh
- net Self_RX renamed Self_RXh
- net Self_RXh: no longer R?.1
- net Self_SWDCLK renamed Self_SWDCLKh
- net Self_SWDIO renamed Self_SWDIOh
- net Self_SWO renamed Self_SWOh
- net Self_TX renamed Self_TXh
- net T_VCP_RX renamed T_VCP_RXh
- net T_VCP_RXh: now also J?.13 (Pin_13)
- net T_VCP_TX renamed T_VCP_TXh
- net T_VCP_TXh: now also J?.14 (Pin_14)
- new net: C?.1, R?.1
- new net: D?.1 (K), R?.2
- new net T_NRST_SWDh: J?.12 (Pin_12), R?.1
- new net T_NRST_SWIMh: R?.2
- new net T_SWDCLKh: J?.6 (Pin_6), R?.1
- new net T_SWDIOh: J?.4 (Pin_4), R?.1
- new net T_SWIMh: R?.2
- new net T_SWOh: J?.8 (Pin_8), R?.1
- new net T_Vref_SWDh: D?.2 (A), J?.3 (Pin_3), R?.1
- no-connect marks 10 -> 14
Other:
- moved on the sheet: C?, R?, SW?
