File: project files/stlink.sch (KiCad schematic (older format))
At the start: 63 parts

Commit message: minor tracing
Parts:
- removed J?: Side Connectors, Package_DIP:DIP-28_W15.24mm_Socket, symbol Connector_Generic:Conn_02x14_Counter_Clockwise
- added J3: Self, Connector_PinHeader_2.54mm:PinHeader_1x14_P2.54mm_Vertical, symbol Connector_Generic:Conn_01x14
- added J5: Target, Connector_PinHeader_2.54mm:PinHeader_1x14_P2.54mm_Vertical, symbol Connector_Generic:Conn_01x14
- added U2: STM32F103CBUx, Package_DFN_QFN:QFN-48-1EP_7x7mm_P0.5mm_EP5.6x5.6mm, symbol MCU_ST_STM32F1:STM32F103CBUx
- gave numbers to parts that had none: 62
Connections:
- net labels added: Board_ID
- wire segments 179 -> 208
- no-connect marks 17 -> 26
Other:
- note added: "Added for possibility to use different package.\nSolder one microcontroller only."
- note added: "Board ID"
- note added: "KA-NUCLEO-F411CE uses STM32F103CBU6 as STLink\nGreen Pill uses STM32F103CBT6 as Black Magic Probe\nSpeedy uses STM32F103C8T6 as STLink v2.1"
- note added: "Original boards use as ST-link V2.1:\n- STM32F103CBT6 : Nucleo 32 boards [STM8 and STM32F]\n- STM32F103CBT6TR : Nucleo 64 boards with STM8\nOriginal boards use as ST-Link V2:\n- STM32F103C8T6 : F4Discovery\nSTLink clones use STM32F101****"
- note removed: "Original boards use as ST-link V2.1:\n- STM32F103CBT6 : Nucleo 32 boards [STM8 and STM32F]\n- STM32F103CBT6TR : Nucleo 64 boards with STM8\n\nOriginal boards use as ST-Link V2:\n- STM32F103C8T6 : F4Discovery\n\nClones use STM32F101****\n\nKA-NUCLEO-F411CE uses:\n- STM32F103CBU6"
- moved on the sheet: C10, C11, C13, C14, C15, C3, C4, C5, C6, C7, D4, R14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

Commit message: new references
Parts:
- C1, C11, C12, C13, C15, C16, C2, C3, C4, C5, C6, C7, C8, C9: footprint Capacitor_SMD:C_0805_2012Metric -> Capacitor_SMD:C_0603_1608Metric
- R1, R10, R11, R12, R13, R14, R15, R16, R17, R18, R19, R2, R20, R21, R22, R23, R24, R25, R26, R27, R28, R29, R3, R30, R31, R32, R33, R34, R4, R5, R6, R7, R8, R9: footprint Resistor_SMD:R_0805_2012Metric -> Resistor_SMD:R_0603_1608Metric
Connections:
- net BOOT_0(h): now also C11.2; no longer C11.1
- net GNDD: now also C11.1, C12.1; no longer C11.2, C12.2
- net Self_NRST(h): now also C12.2; no longer C12.1
Other:
- note added: "KA-NUCLEO-F411CE uses STM32F103CBU6 as STLink\nGreen Pill uses STM32F103CBT6 as Black Magic Probe\nSpeedy uses STM32F103C8T6 as STLink v2.1\n\nSTM32+MSD+VCP or STM32+AUDIO can be done with STM32F1xxCBxx\nOther wise: "The up-to-date firmware is too big for this board""
- note added: "MMBT9013 (SOT-23) is pinout compatible with:\n- MMBT2222\n- MMBT3904 (Maple Mini, marking 1AM)\n- BC847\n"
- note added: "Original boards use as ST-link V2.1:\n- STM32F103CBT6 : Nucleo 32 boards [STM8 and STM32F]\n- STM32F103CBT6TR : Nucleo 64 boards with STM8\nOriginal boards use as ST-Link V2:\n- STM32F103C8T6 : F4Discovery\nSTLink clones use STM32F101****\nSome clones use CKS32F103C8xx"
- note added: "Reset"
- note added: "Second microcontroller is added for possibility to use different package.\nSolder one microcontroller only."
- note added: "or SS14\nor PMEG2010\nor MBR130"
- note removed: "Added for possibility to use different package.\nSolder one microcontroller only."
- note removed: "KA-NUCLEO-F411CE uses STM32F103CBU6 as STLink\nGreen Pill uses STM32F103CBT6 as Black Magic Probe\nSpeedy uses STM32F103C8T6 as STLink v2.1"
- note removed: "MMBT9013 (SOT-23) is pinout compatible with:\n- MMBT2222\n- MMBT3904\n- BC847\n"
- note removed: "Original boards use as ST-link V2.1:\n- STM32F103CBT6 : Nucleo 32 boards [STM8 and STM32F]\n- STM32F103CBT6TR : Nucleo 64 boards with STM8\nOriginal boards use as ST-Link V2:\n- STM32F103C8T6 : F4Discovery\nSTLink clones use STM32F101****"
- note removed: "Reset Circuit"
- note removed: "or SS14\nor PMEG2010"
- moved on the sheet: C11, C12, R14, R15, R16
