File: project files/stlink.sch (KiCad schematic (older format))
At the start: 65 parts, among them J1 USB Type C, J2 Power Target, J3 Self, J4 STDC-14, J5 Target, Q1 MMBT9013, U1 STM32F103CBTx, U2 STM32F103CBUx, U3 AMS1117-3.3, Y1 8MHz

Commit message: Update stlink.sch
Connections:
- wire segments 208 -> 201
Other:
- note added: "KA-NUCLEO-F411CE uses STM32F103CBU6 as STLink\nGreen Pill uses STM32F103CBT6 as Black Magic Probe\nSpeedy uses STM32F103C8T6 as STLink v2.1\n\nSTM32+MSD+VCP or STM32+AUDIO can be done with STM32F1xxCBxx only!\nOther wise: "The up-to-date firmware is too big for this board""
- note added: "MMBT9013 (SOT-23) is pinout compatible with:\n- MMBT2222 (STM8 Nucleo32)\n- MMBT3904 (Maple Mini, marking 1AM)\n- BC847\n"
- note added: "Right side is from\nSTLink v3 (MB1440B)"
- note removed: "KA-NUCLEO-F411CE uses STM32F103CBU6 as STLink\nGreen Pill uses STM32F103CBT6 as Black Magic Probe\nSpeedy uses STM32F103C8T6 as STLink v2.1\n\nSTM32+MSD+VCP or STM32+AUDIO can be done with STM32F1xxCBxx\nOther wise: "The up-to-date firmware is too big for this board""
- note removed: "MMBT9013 (SOT-23) is pinout compatible with:\n- MMBT2222\n- MMBT3904 (Maple Mini, marking 1AM)\n- BC847\n"
- moved on the sheet: C10, C11, C12, C13, C14, C15, C7, C8, C9, D2, D4, R12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

Commit message: added reference for BMP
Parts:
- removed R4, R8: 10R, Resistor_SMD:R_0603_1608Metric, symbol Device:R
Other:
- note added: "Just in case to convert into\nBlack Magic Probe"
- note added: "KA-NUCLEO-F411CE uses STM32F103CBU6 as STLink\nGreen Pill uses STM32F103CBT6 as Black Magic Probe\nSpeedy uses STM32F103C8T6 as STLink v2.1\nBlack Magic Probe 2.1 uses STM32F103BBU6\nSTM32+MSD +VCP or STM32+AUDIO can be done with STM32F1xxCBxx only!\nOther wise: "The up-to-date firmware is too big for this board""
- note added: "Pinout of right side is like on\nSTLink v3 (MB1440B)"
- note removed: "KA-NUCLEO-F411CE uses STM32F103CBU6 as STLink\nGreen Pill uses STM32F103CBT6 as Black Magic Probe\nSpeedy uses STM32F103C8T6 as STLink v2.1\n\nSTM32+MSD+VCP or STM32+AUDIO can be done with STM32F1xxCBxx only!\nOther wise: "The up-to-date firmware is too big for this board""
- note removed: "Right side is from\nSTLink v3 (MB1440B)"
Changed lines of the file:
@@
 Rev ""
 Comp ""
-Comment1 "For SWD / SWIM / VCP isolation consided ISO7231 or ISO764xFM"
+Comment1 "For SWD/SWIM/VCP isolation consided ISO7231 or ISO764xFM"
 Comment2 "For USB isolation consider Si8606AC-B-IS1 or ADuM5000/5001 or ADuM1200/1201"
-Comment3 "For ESD protection of SWD / SWIM / VCP consider ESDA6V1BC6"
+Comment3 "For ESD protection of SWD/SWIM/VCP consider ESDA6V1BC6, of TXS0108E for level shifting"
 Comment4 "For ESD protection of USB consider NUP2201 or USBLC6-2P6"
 $EndDescr
@@
 Wire Wire Line
 	2600 6650 2450 6650
-$Comp
-L Device:R R4
-U 1 1 5E5B2510
-P 2750 6650
-F 0 "R4" V 2700 6500 50  0000 C CNN
-F 1 "10R" V 2750 6650 50  0000 C CNN
-F 2 "Resistor_SMD:R_0603_1608Metric" V 2680 6650 50  0001 C CNN
-F 3 "~" H 2750 6650 50  0001 C CNN
-	1    2750 6650
-	0    1    1    0
-$EndComp
-Wire Wire Line
-	2950 6750 2450 6750
-$Comp
-L Device:R R8
-U 1 1 5E55F0CC
-P 3100 6750
-F 0 "R8" V 3050 6600 50  0000 C CNN
-F 1 "10R" V 3100 6750 50  0000 C CNN
-F 2 "Resistor_SMD:R_0603_1608Metric" V 3030 6750 50  0001 C CNN
-F 3 "~" H 3100 6750 50  0001 C CNN
-	1    3100 6750
-	0    1    1    0
-$EndComp
 NoConn ~ 1150 5850
 Text Label 1150 7150 2    50   ~ 0
@@
 T_SWDCLK
 NoConn ~ 2450 6550
-Text Label 2900 6650 0    50   ~ 0
+Text Label 2600 6650 0    50   ~ 0
 STLINK_LED
 Text Label 1150 5750 2    50   ~ 0
@@
 Text Label 1150 6950 2    50   ~ 0
 T_SWDIO_IN
-Text Label 3250 6750 0    50   ~ 0
+Text Label 2600 6750 0    50   ~ 0
 T_SWO
 Text Label 2450 7250 0    50   ~ 0
@@
 	1    0    0    -1
 $EndComp
-Text Notes 750  4350 0    50   ~ 0
+Text Notes 600  4350 0    50   ~ 0
 Original boards use as ST-link V2.1:\n- STM32F103CBT6 : Nucleo 32 boards [STM8 and STM32F]\n- STM32F103CBT6TR : Nucleo 64 boards with STM8\nOriginal boards use as ST-Link V2:\n- STM32F103C8T6 : F4Discovery\nSTLink clones use STM32F101****\nSome clones use CKS32F103C8xx
 Text Notes 9350 1000 0    50   ~ 0
@@
 Text GLabel 10350 3800 2    50   Input ~ 0
 T_SWIM(h)
-Text Notes 9100 2650 0    100  Italic 20
+Text Notes 9400 2650 0    100  Italic 20
 Side Connectors
 Text GLabel 10350 3500 2    50   Input ~ 0
@@
 	1    0    0    -1
 $EndComp
-Text Notes 3050 4350 0    50   ~ 0
-KA-NUCLEO-F411CE uses STM32F103CBU6 as STLink\nGreen Pill uses STM32F103CBT6 as Black Magic Probe\nSpeedy uses STM32F103C8T6 as STLink v2.1\n\nSTM32+MSD+VCP or STM32+AUDIO can be done with STM32F1xxCBxx only!\nOther wise: "The up-to-date firmware is too big for this board"
+Text Notes 2950 4350 0    50   ~ 0
+KA-NUCLEO-F411CE uses STM32F103CBU6 as STLink\nGreen Pill uses STM32F103CBT6 as Black Magic Probe\nSpeedy uses STM32F103C8T6 as STLink v2.1\nBlack Magic Probe 2.1 uses STM32F103BBU6\nSTM32+MSD +VCP or STM32+AUDIO can be done with STM32F1xxCBxx only!\nOther wise: "The up-to-date firmware is too big for this board"
 Wire Wire Line
 	2950 5000 3350 5000
@@
 STLINK_LED
 $Comp
-L power:GNDD #PWR?
+L power:GNDD #PWR0101
 U 1 1 5ED115B2
 P 6500 1050
-F 0 "#PWR?" H 6500 800 50  0001 C CNN
+F 0 "#PWR0101" H 6500 800 50  0001 C CNN
 F 1 "GNDD" H 6504 895 50  0000 C CNN
 F 2 "" H 6500 1050 50  0001 C CNN
@@
 $EndComp
 $Comp
-L power:+3V3 #PWR?
+L power:+3V3 #PWR0102
 U 1 1 5ED11C16
 P 5700 750
-F 0 "#PWR?" H 5700 600 50  0001 C CNN
+F 0 "#PWR0102" H 5700 600 50  0001 C CNN
 F 1 "+3V3" H 5715 923 50  0000 C CNN
 F 2 "" H 5700 750 50  0001 C CNN
@@
 Text Notes 5900 3750 0    100  Italic 20
 HSE
-Text Notes 10100 4550 0    50   ~ 0
-Right side is from\nSTLink v3 (MB1440B)
+Text Notes 10050 4550 0    50   ~ 0
+Pinout of right side is like on\nSTLink v3 (MB1440B)
 Wire Wire Line
 	3350 5400 3350 5000
 Connection ~ 3350 5000
+Wire Wire Line
+	2600 6750 2450 6750
+Text Notes 9950 4550 2    50   ~ 0
+Just in case to convert into\nBlack Magic Probe
 $EndSCHEMATC

Commit message: Update stlink.sch
Parts:
- removed U2: STM32F103CBUx, Package_DFN_QFN:QFN-48-1EP_7x7mm_P0.5mm_EP5.6x5.6mm, symbol MCU_ST_STM32F1:STM32F103CBUx
- added U?: STM32F103CBUx, Package_DFN_QFN:QFN-48-1EP_7x7mm_P0.5mm_EP5.6x5.6mm, symbol MCU_ST_STM32F1:STM32F103CBUx
Changed lines of the file:
@@
 Text Label 1150 5350 2    50   ~ 0
 Board_ID
-$Comp
-L MCU_ST_STM32F1:STM32F103CBUx U2
-U 1 1 5EA01F43
-P 4700 5950
-F 0 "U2" H 5000 4400 50  0000 C CNN
-F 1 "STM32F103CBUx" H 5250 4500 50  0000 C CNN
-F 2 "Package_DFN_QFN:QFN-48-1EP_7x7mm_P0.5mm_EP5.6x5.6mm" H 4100 4550 50  0001 R CNN
-F 3 "http://www.st.com/st-web-ui/static/active/en/resource/technical/document/datasheet/CD00161566.pdf" H 4700 5950 50  0001 C CNN
-	1    4700 5950
-	1    0    0    -1
-$EndComp
-Text Label 4000 4650 2    50   ~ 0
-STLINK_NRST
-Wire Wire Line
-	4900 4450 4900 4400
-Wire Wire Line
-	4900 4400 4800 4400
-Wire Wire Line
-	4800 4450 4800 4400
-Connection ~ 4800 4400
-Wire Wire Line
-	4800 4400 4700 4400
-Wire Wire Line
-	4700 4450 4700 4400
-Connection ~ 4700 4400
-Wire Wire Line
-	4700 4400 4600 4400
-Wire Wire Line
-	4600 4450 4600 4400
-Connection ~ 4600 4400
-Wire Wire Line
-	4600 4400 4500 4400
-Wire Wire Line
-	4500 4450 4500 4400
-Wire Wire Line
-	4900 7500 4900 7450
-Wire Wire Line
-	4800 7450 4800 7500
-Connection ~ 4800 7500
-Wire Wire Line
-	4800 7500 4900 7500
-Wire Wire Line
-	4700 7450 4700 7500
-Connection ~ 4700 7500
-Wire Wire Line
-	4700 7500 4800 7500
-Wire Wire Line
-	4600 7450 4600 7500
-Connection ~ 4600 7500
-Wire Wire Line
-	4600 7500 4700 7500
-Wire Wire Line
-	4500 7450 4500 7500
-Wire Wire Line
-	4500 7500 4600 7500
-Text Label 4000 4850 2    50   ~ 0
-BOOT_0
-Text Label 4000 5050 2    50   ~ 0
-STLINK_OSC_IN
-Text Label 4000 5150 2    50   ~ 0
-STLINK_OST_OUT
-Text Label 4000 5350 2    50   ~ 0
-Board_ID
-NoConn ~ 4000 5450
-NoConn ~ 4000 5550
-NoConn ~ 4000 5850
-NoConn ~ 4000 6150
-NoConn ~ 4000 7250
-NoConn ~ 5300 5850
-NoConn ~ 5300 6150
-NoConn ~ 5300 6350
-NoConn ~ 5300 6550
-Text Label 5300 6650 0    50   ~ 0
-TX
-Text Label 5300 6750 0    50   ~ 0
-RX
-Text Label 5300 6850 0    50   ~ 0
-STLINK_USB_D-
-Text Label 5300 7250 0    50   ~ 0
-USB_RENUMn
-Text Label 5300 6950 0    50   ~ 0
-STLINK_USB_D+
-Text Label 5300 7150 0    50   ~ 0
-SWDCLK
-Text Label 5300 7050 0    50   ~ 0
-SWDIO
 Wire Wire Line
 	2500 4400 2950 4400
@@
 Wire Wire Line
 	2950 5050 2950 5000
-$Comp
-L power:GNDD #PWR019
-U 1 1 5EBA903C
-P 4900 7550
-F 0 "#PWR019" H 4900 7300 50  0001 C CNN
-F 1 "GNDD" H 4904 7395 50  0000 C CNN
-F 2 "" H 4900 7550 50  0001 C CNN
-F 3 "" H 4900 7550 50  0001 C CNN
-	1    4900 7550
-	1    0    0    -1
-$EndComp
-Wire Wire Line
-	4900 7550 4900 7500
-Connection ~ 4900 7500
-Text Label 4000 5750 2    50   ~ 0
-T_NRST_SWD
-Text Label 4000 5950 2    50   ~ 0
-BOOT_1
-Text Label 4000 6050 2    50   ~ 0
-SWO
-Text Label 4000 7150 2    50   ~ 0
-T_SWDIO
-Text Label 4000 7050 2    50   ~ 0
-T_SWDCLK
-Text Label 4000 6250 2    50   ~ 0
-T_NRST_SWIM_IN
-Text Label 4000 6350 2    50   ~ 0
-T_NRST_SWIM
-Text Label 4000 6450 2    50   ~ 0
-T_SWIM_IN
-Text Label 4000 6550 2    50   ~ 0
-T_SWIM
-Text Label 4000 6650 2    50   ~ 0
-T_SWIM_IN
-Text Label 4000 6850 2    50   ~ 0
-T_SWIM
-Text Label 4000 6750 2    50   ~ 0
-T_SWIM_IN
-Text Label 4000 6950 2    50   ~ 0
-T_SWDIO_IN
-Text Label 5300 6250 0    50   ~ 0
-T_SWDCLK
-Text Label 5300 6050 0    50   ~ 0
-STLINK_RX
-Text Label 5300 5950 0    50   ~ 0
-STLINK_TX
-Text Label 5300 5750 0    50   ~ 0
-AIN
-Text Label 5300 6450 0    50   ~ 0
-T_JTDI
-Text Notes 1850 7700 0    50   Italic 10
-Second microcontroller is added for possibility to use different package.\nSolder one microcontroller only.
 Wire Wire Line
 	2950 4400 3350 4400
@@
 	3350 4400 3350 5000
 Connection ~ 2950 4400
-Wire Wire Line
-	4500 4400 3350 4400
-Connection ~ 4500 4400
-Connection ~ 3350 4400
 $Comp
 L Connector_Generic:Conn_01x14 J5
@@
 Text Notes 9950 4550 2    50   ~ 0
 Just in case to convert into\nBlack Magic Probe
+Wire Wire Line
+	4900 7500 4900 7450
+Wire Wire Line
+	4800 7450 4800 7500
+Connection ~ 4800 7500
+Wire Wire Line
+	4800 7500 4900 7500
+Wire Wire Line
+	4700 7450 4700 7500
+Connection ~ 4700 7500
+Wire Wire Line
+	4700 7500 4800 7500
+Wire Wire Line
+	4600 7450 4600 7500
+Connection ~ 4600 7500
+Wire Wire Line
+	4600 7500 4700 7500
+Wire Wire Line
+	4500 7450 4500 7500
+Wire Wire Line
+	4500 7500 4600 7500
+$Comp
+L power:GNDD #PWR?
+U 1 1 5EC7BAF8
+P 4900 7550
+F 0 "#PWR?" H 4900 7300 50  0001 C CNN
+F 1 "GNDD" H 4904 7395 50  0000 C CNN
+F 2 "" H 4900 7550 50  0001 C CNN
+F 3 "" H 4900 7550 50  0001 C CNN
+	1    4900 7550
+	1    0    0    -1
+$EndComp
+Wire Wire Line
+	4900 7550 4900 7500
+Connection ~ 4900 7500
+Text Notes 1850 7700 0    50   Italic 10
+Second microcontroller is added for possibility to use different package.\nSolder one microcontroller only.
+Text Label 5300 6450 0    50   ~ 0
+T_JTDI
+Text Label 5300 5750 0    50   ~ 0
+AIN
+Text Label 5300 5950 0    50   ~ 0
+STLINK_TX
+Text Label 5300 6050 0    50   ~ 0
+STLINK_RX
+Text Label 5300 6250 0    50   ~ 0
+T_SWDCLK
+Text Label 4000 6950 2    50   ~ 0
+T_SWDIO_IN
+Text Label 4000 6750 2    50   ~ 0
+T_SWIM_IN
+Text Label 4000 6850 2    50   ~ 0
+T_SWIM
+Text Label 4000 6650 2    50   ~ 0
+T_SWIM_IN
+Text Label 4000 6550 2    50   ~ 0
+T_SWIM
+Text Label 4000 6450 2    50   ~ 0
+T_SWIM_IN
+Text Label 4000 6350 2    50   ~ 0
+T_NRST_SWIM
+Text Label 4000 6250 2    50   ~ 0
+T_NRST_SWIM_IN
+Text Label 4000 7050 2    50   ~ 0
+T_SWDCLK
+Text Label 4000 7150 2    50   ~ 0
+T_SWDIO
+Text Label 4000 6050 2    50   ~ 0
+SWO
+Text Label 4000 5950 2    50   ~ 0
+BOOT_1
+Text Label 4000 5750 2    50   ~ 0
+T_NRST_SWD
+Text Label 5300 7050 0    50   ~ 0
+SWDIO
+Text Label 5300 7150 0    50   ~ 0
+SWDCLK
+Text Label 5300 6950 0    50   ~ 0
+STLINK_USB_D+
+Text Label 5300 7250 0    50   ~ 0
+USB_RENUMn
+Text Label 5300 6850 0    50   ~ 0
+STLINK_USB_D-
+Text Label 5300 6750 0    50   ~ 0
+RX
+Text Label 5300 6650 0    50   ~ 0
+TX
+NoConn ~ 5300 6550
+NoConn ~ 5300 6350
+NoConn ~ 5300 6150
+NoConn ~ 5300 5850
+NoConn ~ 4000 7250
+NoConn ~ 4000 6150
+NoConn ~ 4000 5850
+NoConn ~ 4000 5550
+NoConn ~ 4000 5450
+Text Label 4000 5350 2    50   ~ 0
+Board_ID
+Text Label 4000 5150 2    50   ~ 0
+STLINK_OST_OUT
+Text Label 4000 5050 2    50   ~ 0
+STLINK_OSC_IN
+Text Label 4000 4850 2    50   ~ 0
+BOOT_0
+Wire Wire Line
+	4500 4450 4500 4400
+Wire Wire Line
+	4600 4400 4500 4400
+Connection ~ 4600 4400
+Wire Wire Line
+	4600 4450 4600 4400
+Wire Wire Line
+	4700 4400 4600 4400
+Connection ~ 4700 4400
+Wire Wire Line
+	4700 4450 4700 4400
+Wire Wire Line
+	4800 4400 4700 4400
+Connection ~ 4800 4400
+Wire Wire Line
+	4800 4450 4800 4400
+Wire Wire Line
+	4900 4400 4800 4400
+Wire Wire Line
+	4900 4450 4900 4400
+Text Label 4000 4650 2    50   ~ 0
+STLINK_NRST
+$Comp
+L MCU_ST_STM32F1:STM32F103CBUx U?
+U 1 1 5EC7BB3B
+P 4700 5950
+F 0 "U?" H 5000 4400 50  0000 C CNN
+F 1 "STM32F103CBUx" H 5250 4500 50  0000 C CNN
+F 2 "Package_DFN_QFN:QFN-48-1EP_7x7mm_P0.5mm_EP5.6x5.6mm" H 4100 4550 50  0001 R CNN
+F 3 "http://www.st.com/st-web-ui/static/active/en/resource/technical/document/datasheet/CD00161566.pdf" H 4700 5950 50  0001 C CNN
+	1    4700 5950
+	1    0    0    -1
+$EndComp
+Wire Wire Line
+	4500 4400 3350 4400
+Connection ~ 4500 4400
+Connection ~ 3350 4400
 $EndSCHEMATC

Commit message: multi-sheet introduction for spare parts
Parts:
- removed J3: Self, Connector_PinHeader_2.54mm:PinHeader_1x14_P2.54mm_Vertical, symbol Connector_Generic:Conn_01x14
- removed J4: STDC-14, Connector_PinHeader_1.27mm:PinHeader_2x07_P1.27mm_Vertical_SMD, symbol Connector_Generic:Conn_02x07_Odd_Even
- added J4: Target STDC-14, Connector_PinHeader_1.27mm:PinHeader_2x07_P1.27mm_Vertical, symbol Connector:Conn_ST_STDC14
- added J6: Self, Connector_PinHeader_1.27mm:PinHeader_2x07_P1.27mm_Vertical_SMD, symbol Connector:Conn_ST_STDC14
- gave numbers to parts that had none: 1
Connections:
- wire segments 201 -> 194
- no-connect marks 26 -> 25
Other:
- note added: "Self\nProgramming"
- note added: "Target Programming Connectors"
- note removed: "STDC-14 as JTAG \nor SWD+VCP"
- note removed: "Side Connectors"

Commit message: some rerouting
Parts:
- removed R22: 220R, Resistor_SMD:R_0603_1608Metric, symbol Device:R
- removed R25: 680R, Resistor_SMD:R_0603_1608Metric, symbol Device:R
- removed U2: STM32F103CBUx, Package_DFN_QFN:QFN-48-1EP_7x7mm_P0.5mm_EP5.6x5.6mm, symbol MCU_ST_STM32F1:STM32F103CBUx
- added R?: 680R, Resistor_SMD:R_0603_1608Metric, symbol Device:R
- added R?: 220R, Resistor_SMD:R_0603_1608Metric, symbol Device:R
- renumbered C8 to C10, C14 to C11, C11 to C13, C15 to C14, C9 to C15, C10 to C8, C13 to C9, D4 to D3, D3 to D4, J5 to J2, J2 to J3, J6 to J4, J4 to J5, R13 to R10, R12 to R11, R16 to R12, R14 to R13, R15 to R14, R18 to R15, R17 to R16, R19 to R17, R20 to R18, R21 to R19, R23 to R21, R24 to R22, R26 to R24, R27 to R25, R28 to R26, R29 to R27, R30 to R28, R31 to R29, R32 to R30, R33 to R31, R34 to R32, R5 to R4, R6 to R5, R7 to R6, R9 to R7, R10 to R8, R11 to R9, U3 to U2
Connections:
- net labels added: OSC_IN, OSC_OUT, SELF_NRST
- net labels removed: STLINK_NRST, STLINK_OSC_IN, STLINK_OST_OUT
- wire segments 194 -> 168
- no-connect marks 25 -> 16
Other:
- note removed: "Second microcontroller is added for possibility to use different package.\nSolder one microcontroller only."
- moved on the sheet: C3, C4, C5, C6, C7, R21, R22, U1

Commit message: fixes
Parts:
- added R?: 100, Resistor_SMD:R_0603_1608Metric, symbol Device:R
Connections:
- wire segments 168 -> 169
Changed lines of the file:
@@
 L power:GNDD #PWR045
 U 1 1 5EC39966
-P 9850 2250
-F 0 "#PWR045" H 9850 2000 50  0001 C CNN
-F 1 "GNDD" H 9854 2095 50  0000 C CNN
-F 2 "" H 9850 2250 50  0001 C CNN
-F 3 "" H 9850 2250 50  0001 C CNN
-	1    9850 2250
+P 9950 2200
+F 0 "#PWR045" H 9950 1950 50  0001 C CNN
+F 1 "GNDD" H 9954 2045 50  0000 C CNN
+F 2 "" H 9950 2200 50  0001 C CNN
+F 3 "" H 9950 2200 50  0001 C CNN
+	1    9950 2200
 	1    0    0    -1
 $EndComp
@@
 Wire Wire Line
 	10050 2900 10050 2950
-Wire Wire Line
-	9950 2200 9950 2250
-Wire Wire Line
-	9950 2250 9850 2250
-Wire Wire Line
-	9850 2200 9850 2250
-Connection ~ 9850 2250
 Text GLabel 10550 6450 2    50   Output ~ 0
 T_VCP_RX(h)
@@
 F1 "spare connectivity.sch" 50
 $EndSheet
-Text GLabel 5500 1000 0    50   BiDi ~ 0
+Text GLabel 5550 1000 0    50   BiDi ~ 0
 STLINK_LED
 Text GLabel 6750 800  2    50   BiDi ~ 0
@@
 Wire Wire Line
 	3850 6750 3800 6750
+Wire Wire Line
+	3850 6400 3850 6300
+Wire Wire Line
+	3850 6700 3850 6750
+Connection ~ 3850 6750
+$Comp
+L Device:R R?
+U 1 1 5EF8AF16
+P 9650 2250
+F 0 "R?" V 9550 2250 50  0000 C CNN
+F 1 "100" V 9650 2250 50  0000 C CNN
+F 2 "Resistor_SMD:R_0603_1608Metric" V 9580 2250 50  0001 C CNN
+F 3 "~" H 9650 2250 50  0001 C CNN
+	1    9650 2250
+	0    1    -1   0
+$EndComp
+$Comp
+L power:GNDD #PWR?
+U 1 1 5EF8B5FE
+P 9500 2250
+F 0 "#PWR?" H 9500 2000 50  0001 C CNN
+F 1 "GNDD" H 9504 2095 50  0000 C CNN
+F 2 "" H 9500 2250 50  0001 C CNN
+F 3 "" H 9500 2250 50  0001 C CNN
+	1    9500 2250
+	1    0    0    -1
+$EndComp
+Wire Wire Line
+	9800 2250 9850 2250
+Wire Wire Line
+	9850 2250 9850 2200
 $EndSCHEMATC

Commit message: updates with level converters
Parts:
- removed C2: 1nF, Capacitor_SMD:C_0603_1608Metric, symbol Device:C
- removed J2: Target, Connector_PinHeader_2.54mm:PinHeader_1x14_P2.54mm_Vertical, symbol Connector_Generic:Conn_01x14
- removed J4: Self, Connector_PinHeader_1.27mm:PinHeader_2x07_P1.27mm_Vertical_SMD, symbol Connector:Conn_ST_STDC14
- removed R24: 47R, Resistor_SMD:R_0603_1608Metric, symbol Device:R
- removed R26, R27, R28, R29, R30, R31, R32, R5, R6: 22R, Resistor_SMD:R_0603_1608Metric, symbol Device:R
- removed R?: 100, Resistor_SMD:R_0603_1608Metric, symbol Device:R
- added J?: SWD, symbol Connector_Generic:Conn_01x06
- added J?: SWIM+VCP, symbol Connector_Generic:Conn_01x06
- added U?: USBLC6-2P6, Package_TO_SOT_SMD:SOT-666, symbol Power_Protection:USBLC6-2P6
- added U?: TXS0108EPW, Package_SO:TSSOP-20_4.4x6.5mm_P0.65mm, symbol Logic_LevelTranslator:TXS0108EPW
- J5: value Target STDC-14 -> STDC-14
Connections:
- net labels removed: +5V
- wire segments 169 -> 154
- no-connect marks 16 -> 12
Other:
- note added: "Target Voltage Detection or power it from STLink"
- note added: "USB Type C as USB 2.0 + VCP and protection"
- note removed: "47R resistors can be 22R"
- note removed: "Just in case to convert into\nBlack Magic Probe"
- note removed: "Pinout of right side is like on\nSTLink v3 (MB1440B)"
- note removed: "SWD/JTAG:"
- note removed: "SWIM:"
- note removed: "Self\nProgramming"
- note removed: "Target Voltage\nDetection or power\nit from STLink"
- note removed: "USB Type C as USB 2.0"
- note removed: "VCP interface"
- moved on the sheet: C10, C11, C12, C13, C14, C15, C16, C8, C9, D1, D2, D3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

Commit message: fix after re-open in last KiCAD
Parts:
- J1: symbol Connector:USB_C_Receptacle_USB2.0 -> stlink-rescue:USB_C_Receptacle_USB2.0-Connector
Changed lines of the file:
@@
 	2250 1100 2250 1050
 $Comp
-L Connector:USB_C_Receptacle_USB2.0 J1
+L stlink-rescue:USB_C_Receptacle_USB2.0-Connector J1
 U 1 1 5E141D2F
 P 950 1700
