File: project files/simplified/stlink.sch (KiCad schematic (older format))
At the start: 56 parts, among them J1 Power Target, J2 USB Type C, J3 SWD, J4 STDC-14, J5 SWIM+VCP, Q1 MMBT9013, U1 AMS1117-3.3, U2 STM32F103CBTx, Y1 8MHz

Commit message: STDC adapters
Changed lines of the file:
@@
 Wire Notes Line
 	6950 5050 11200 5050
-Text GLabel 8700 4400 0    50   Output ~ 0
-GND_detect(h)
-Text GLabel 9250 4350 2    50   Output ~ 0
-GND_detect(h)
-$Comp
-L power:GNDD #PWR036
-U 1 1 5E9AED9E
-P 9100 4400
-F 0 "#PWR036" H 9100 4150 50  0001 C CNN
-F 1 "GNDD" H 9104 4245 50  0000 C CNN
-F 2 "" H 9100 4400 50  0001 C CNN
-F 3 "" H 9100 4400 50  0001 C CNN
-	1    9100 4400
-	-1   0    0    -1
-$EndComp
 $Comp
 L power:GNDD #PWR031
@@
 $EndComp
 Wire Wire Line
-	9250 4350 9100 4350
-Wire Wire Line
-	9100 4350 9100 4400
-Wire Wire Line
 	8100 1100 7850 1100
 Connection ~ 7850 1100
@@
 Wire Wire Line
 	5300 2400 5450 2400
-Wire Wire Line
-	8700 4400 8750 4400
 Wire Wire Line
 	8750 4400 8750 4350
@@
 Wire Wire Line
 	4100 7150 4100 7250
+Wire Wire Line
+	8750 4400 8850 4400
+Connection ~ 8850 4400
 $EndSCHEMATC

Commit message: Fixes
Parts:
- removed J1: Power Target, Connector_PinHeader_2.54mm:PinHeader_2x02_P2.54mm_Vertical, symbol Connector_Generic:Conn_02x02_Odd_Even
- added SW?: Power Ext, symbol Switch:SW_Push_SPDT
Connections:
- net +3V3: now also SW?.1 (A)
- net T_Vref: now also SW?.2 (B)
- net SELF_NRST renamed Self_NRST
- no-connect marks 13 -> 14
Changed lines of the file:
@@
 $EndComp
-Wire Wire Line
-	5400 1300 5450 1300
 Wire Wire Line
 	5450 1350 5450 1300
@@
 Text Notes 5550 1500 0    50   ~ 0
 or:\n1N5817
-Text Notes 4650 1600 0    50   ~ 0
+Text Notes 4650 1800 0    50   ~ 0
 Vref PullDown\ncan be 10K
 $Comp
@@
 Power Regulator
 Wire Wire Line
-	4900 1200 4850 1200
-Wire Wire Line
-	4850 1200 4850 1150
-Wire Wire Line
-	4900 1300 4650 1300
-Wire Wire Line
-	4650 1300 4650 1150
+	4750 1200 4750 1150
 $Comp
 L power:+3V3 #PWR07
 U 1 1 5EA68D52
-P 4850 1150
-F 0 "#PWR07" H 4850 1000 50  0001 C CNN
-F 1 "+3V3" H 4865 1323 50  0000 C CNN
-F 2 "" H 4850 1150 50  0001 C CNN
-F 3 "" H 4850 1150 50  0001 C CNN
-	1    4850 1150
-	1    0    0    -1
-$EndComp
-$Comp
-L Connector_Generic:Conn_02x02_Odd_Even J1
-U 1 1 5E9AB85E
-P 5100 1200
-F 0 "J1" H 5150 1417 50  0000 C CNN
-F 1 "Power Target" H 5150 1326 50  0000 C CNN
-F 2 "Connector_PinHeader_2.54mm:PinHeader_2x02_P2.54mm_Vertical" H 5100 1200 50  0001 C CNN
-F 3 "~" H 5100 1200 50  0001 C CNN
-	1    5100 1200
-	1    0    0    -1
-$EndComp
-Wire Wire Line
-	5400 1200 5450 1200
-Wire Wire Line
-	5450 1200 5450 1300
-Connection ~ 5450 1200
+P 4750 1150
+F 0 "#PWR07" H 4750 1000 50  0001 C CNN
+F 1 "+3V3" H 4765 1323 50  0000 C CNN
+F 2 "" H 4750 1150 50  0001 C CNN
+F 3 "" H 4750 1150 50  0001 C CNN
+	1    4750 1150
+	1    0    0    -1
+$EndComp
 Wire Notes Line
 	7300 2450 11150 2450
@@
 STLINK_LED
 Text GLabel 4050 7150 0    50   Input ~ 0
-SELF_NRST
+Self_NRST
 Text GLabel 7750 5450 0    50   Input ~ 0
-SELF_NRST
+Self_NRST
 Text GLabel 6450 1300 2    50   Input ~ 0
 AIN
@@
 Board_ID
 Text GLabel 1150 4000 0    50   Input ~ 0
-SELF_NRST
+Self_NRST
 Text GLabel 1150 4200 0    50   Input ~ 0
 BOOT_0
@@
 $EndComp
 $Comp
-L power:VBUS #PWR06
-U 1 1 5F215625
-P 4650 1150
-F 0 "#PWR06" H 4650 1000 50  0001 C CNN
-F 1 "VBUS" H 4665 1323 50  0000 C CNN
-F 2 "" H 4650 1150 50  0001 C CNN
-F 3 "" H 4650 1150 50  0001 C CNN
-	1    4650 1150
-	1    0    0    -1
-$EndComp
-$Comp
 L Connector_Generic:Conn_01x06 J3
 U 1 1 5F2190BA
@@
 Wire Wire Line
 	5400 850  5450 850
-Wire Wire Line
-	5450 850  5450 1200
 Wire Wire Line
 	6150 1300 6400 1300
@@
 	8750 4400 8850 4400
 Connection ~ 8850 4400
+Text GLabel 800  5300 0    50   Input ~ 0
+BOOT_1
+Wire Wire Line
+	5450 850  5450 1300
+Wire Wire Line
+	4750 1200 4900 1200
+Wire Wire Line
+	5300 1300 5450 1300
+$Comp
+L Switch:SW_Push_SPDT SW?
+U 1 1 60705C92
+P 5100 1300
+F 0 "SW?" H 5100 1585 50  0000 C CNN
+F 1 "Power Ext" H 5100 1494 50  0000 C CNN
+F 2 "" H 5100 1300 50  0001 C CNN
+F 3 "~" H 5100 1300 50  0001 C CNN
+	1    5100 1300
+	-1   0    0    -1
+$EndComp
+NoConn ~ 4900 1400
 $EndSCHEMATC
