File: project files/simplified/stlink.kicad_pcb (KiCad board)
At the start: 2 copper layers, 43.2 x 17.8 mm, 60 parts, among them J1 Power Target, J2 USB Type C, J3 SWD, J4 STDC-14, J5 SWIM+VCP, J6 Self, J7 Conn_01x04, J8 Conn_01x04, Q1 MMBT9013, U1 AMS1117-3.3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

Commit message: Self RX/TX fix
Connections:
- J6 pad 13: Self_RX(h) -> STLINK_LED
- J6 pad 14: STLINK_LED -> Self_RX(h)

Commit message: STDC adapters
Parts:
- D2: moved to F.Cu
- R13: moved to B.Cu
- moved R1 35.4 mm to (243.7, 93.3)
- moved D2 34.9 mm to (231.1, 124.5)
- moved R13 31.4 mm to (211.3, 109.2)
- moved JP1 17.2 mm to (213.4, 123.8)
- moved J3 15.2 mm to (236.2, 124.5)
- moved J5 15.2 mm to (248.9, 109.2)
- moved Q1 8.05 mm to (247.0, 94.3), turned to 270 degrees
- moved R8 0.92 mm to (250.4, 93.3)
- moved R6 0.90 mm to (250.4, 91.4)
- moved Y1 0.13 mm to (239.3, 117.5)
Connections:
- net GND_detect(h) renamed GNDD

Commit message: edited labels according to kicad 5.99
Parts:
- removed J1: Power Target, Connector_PinHeader_2.54mm:PinHeader_2x02_P2.54mm_Vertical
- removed R20, R21, R22, R23, R24, R25, R26, R27, R28: 47R, Resistor_SMD:R_0603_1608Metric
- moved R3 59.1 mm to (214.0, 132.1)
- moved R5 55.9 mm to (213.8, 130.2)
- moved R12 51.9 mm to (218.4, 118.1)
- moved R11 46.1 mm to (218.4, 116.2)
- moved Q1 34.5 mm to (218.4, 113.7), turned to 0 degrees
- moved R8 8.53 mm to (255.3, 100.3)
- moved R6 6.15 mm to (254.6, 95.9)
- turned J6 to 180 degrees
Connections:
- C1 pad 2: GNDD -> BOOT_1
- C10 pad 1: GNDD -> BOOT_1
- C10 pad 2: SELF_NRST -> Self_NRST
- C11 pad 1: GNDD -> BOOT_1
- C12 pad 2: GNDD -> BOOT_1
- C13 pad 2: GNDD -> BOOT_1
- C2 pad 2: GNDD -> BOOT_1
- C3 pad 2: GNDD -> BOOT_1
- C4 pad 2: GNDD -> BOOT_1
- C5 pad 2: GNDD -> BOOT_1
- C6 pad 2: GNDD -> BOOT_1
- C7 pad 1: GNDD -> BOOT_1
- C8 pad 2: GNDD -> BOOT_1
- C9 pad 2: GNDD -> BOOT_1
- D3 pad 1: GNDD -> BOOT_1
- J2 pad A1: GNDD -> BOOT_1
- J2 pad A12: GNDD -> BOOT_1
- J2 pad A8: Net-(J2-PadA8) -> unconnected-(J2-PadA8)
- J2 pad B1: GNDD -> BOOT_1
- J2 pad B12: GNDD -> BOOT_1
- J2 pad B8: Net-(J2-PadB8) -> unconnected-(J2-PadB8)
- J2 pad S1: Net-(J2-PadS1) -> BOOT_1
- J3 pad 3: GNDD -> BOOT_1
- J4 pad 1: Net-(J4-Pad1) -> unconnected-(J4-Pad1)
- J4 pad 10: T_JTDI(h) -> T_JTDI
- J4 pad 11: GNDD -> BOOT_1
- J4 pad 2: Net-(J4-Pad2) -> unconnected-(J4-Pad2)
- J4 pad 5: GNDD -> BOOT_1
- J4 pad 7: GNDD -> BOOT_1
- J4 pad 9: Net-(J4-Pad9) -> unconnected-(J4-Pad9)
- J5 pad 3: GNDD -> BOOT_1
- J6 pad 1: Net-(J6-Pad1) -> unconnected-(J6-Pad1)
- J6 pad 10: Net-(J6-Pad10) -> unconnected-(J6-Pad10)
- J6 pad 11: Net-(J6-Pad11) -> unconnected-(J6-Pad11)
- J6 pad 12: SELF_NRST -> Self_NRST
- J6 pad 2: Net-(J6-Pad2) -> unconnected-(J6-Pad2)
- J6 pad 5: GNDD -> BOOT_1
- J6 pad 7: GNDD -> BOOT_1
- J6 pad 9: Net-(J6-Pad9) -> unconnected-(J6-Pad9)
- J7 pad 1: SELF_NRST -> Self_NRST
- J8 pad 4: GNDD -> BOOT_1
- R10 pad 2: GNDD -> BOOT_1
- R19 pad 1: GNDD -> BOOT_1
- R29 pad 2: SELF_NRST -> Self_NRST
- R3 pad 2: GNDD -> BOOT_1
- R30 pad 2: GNDD -> BOOT_1
- R5 pad 2: GNDD -> BOOT_1
- R8 pad 2: GNDD -> BOOT_1
- R9 pad 2: GNDD -> BOOT_1
- U1 pad 1: GNDD -> BOOT_1
- U2 pad 11: Net-(U2-Pad11) -> unconnected-(U2-Pad11)
- U2 pad 14: Net-(U2-Pad14) -> unconnected-(U2-Pad14)
- U2 pad 16: Net-(U2-Pad16) -> unconnected-(U2-Pad16)
- U2 pad 19: Net-(U2-Pad19) -> unconnected-(U2-Pad19)
- U2 pad 20: GNDD -> BOOT_1
- U2 pad 23: GNDD -> BOOT_1
- U2 pad 28: Net-(U2-Pad28) -> unconnected-(U2-Pad28)
- U2 pad 29: Net-(U2-Pad29) -> unconnected-(U2-Pad29)
- U2 pad 3: Net-(U2-Pad3) -> unconnected-(U2-Pad3)
- U2 pad 35: GNDD -> BOOT_1
- U2 pad 4: Net-(U2-Pad4) -> unconnected-(U2-Pad4)
- U2 pad 40: Net-(U2-Pad40) -> unconnected-(U2-Pad40)
- U2 pad 47: GNDD -> BOOT_1
- U2 pad 7: SELF_NRST -> Self_NRST
- U2 pad 8: GNDD -> BOOT_1
- U3 pad 11: Net-(U3-Pad11) -> unconnected-(U3-Pad11)
- U3 pad 14: Net-(U3-Pad14) -> unconnected-(U3-Pad14)
- U3 pad 16: Net-(U3-Pad16) -> unconnected-(U3-Pad16)
- U3 pad 19: Net-(U3-Pad19) -> unconnected-(U3-Pad19)
- U3 pad 23: GNDD -> BOOT_1
- U3 pad 28: Net-(U3-Pad28) -> unconnected-(U3-Pad28)
- U3 pad 29: Net-(U3-Pad29) -> unconnected-(U3-Pad29)
- U3 pad 3: Net-(U3-Pad3) -> unconnected-(U3-Pad3)
- U3 pad 35: GNDD -> BOOT_1
- U3 pad 4: Net-(U3-Pad4) -> unconnected-(U3-Pad4)
- U3 pad 40: Net-(U3-Pad40) -> unconnected-(U3-Pad40)
- U3 pad 47: GNDD -> BOOT_1
- U3 pad 49: GNDD -> BOOT_1
- U3 pad 8: GNDD -> BOOT_1
- Y1 pad 2: GNDD -> BOOT_1
- Y1 pad 4: GNDD -> BOOT_1
Routing:
- net SWO: track 0.00 -> 9.44 mm
- net SWDCLK: track 0.00 -> 7.61 mm
- net SWDIO: track 0.00 -> 6.84 mm
- net Self_RX(h): track 0.00 -> 4.09 mm
- net STLINK_LED: track 0.00 -> 4.09 mm
Other:
- net class Default removed
