File: project files/simplified/stlink.kicad_sch (KiCad schematic)
At the start: 49 parts, among them J2 USB Type C, J3 SWD, J4 STDC-14, J5 SWIM+VCP, Q1 MMBT9013, SW1 Power Ext, U1 AMS1117-3.3, U2 STM32F103CBTx, Y1 8MHz

Commit message: edited labels according to kicad 5.99
Connections:
- net GNDD: now also J2.S1 (SHIELD)
- no-connect marks 14 -> 13
Changed lines of the file:
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@@
-(kicad_sch (version 20210406) (generator eeschema)
+(kicad_sch (version 20210621) (generator eeschema)
   (paper "A4")
   (title_block
@@
   (junction (at 222.25 27.94) (diameter 1.016) (color 0 0 0 0))
   (junction (at 224.79 111.76) (diameter 1.016) (color 0 0 0 0))
-  (no_connect (at 16.51 66.04))
   (no_connect (at 29.21 121.92))
   (no_connect (at 29.21 124.46))
@@
     )
     (property "Datasheet" "" (id 3) (at 259.08 29.21 0)
+      (effects (font (size 1.27 1.27)) hide)
+    )
+    (pin "1")
+  )
+  (symbol (lib_id "power:GNDD") (at 16.51 66.04 0) (unit 1)
+    (in_bom yes) (on_board yes)
+    (property "Reference" "#PWR?" (id 0) (at 16.51 72.39 0)
+      (effects (font (size 1.27 1.27)) hide)
+    )
+    (property "Value" "GNDD" (id 1) (at 16.6116 69.977 0))
+    (property "Footprint" "" (id 2) (at 16.51 66.04 0)
+      (effects (font (size 1.27 1.27)) hide)
+    )
+    (property "Datasheet" "" (id 3) (at 16.51 66.04 0)
       (effects (font (size 1.27 1.27)) hide)
     )
@@
       (reference "#PWR055") (unit 1) (value "GNDD") (footprint "")
     )
+    (path "/8545ec10-b5d1-4259-9ef5-726913246f4b"
+      (reference "#PWR?") (unit 1) (value "GNDD") (footprint "")
+    )
     (path "/00000000-0000-0000-0000-00005e270620"
