File: project files/protected/spare connectivity.sch (KiCad schematic (older format))
At the start: 4 parts, among them J6 Self, J7 Conn_01x04, J8 Conn_01x04, U5 STM32F103CBUx

Commit message: Fixes
Parts:
- renumbered J6 to J5, J7 to J6, J8 to J7, U5 to U6
Connections:
- net MCO: now reaches U6.29 (PA8)
- net Board_ID2: now reaches U6.3 (PC14)
- net Board_ID renamed Board_ID1
- no-connect marks 12 -> 10
Changed lines of the file:
@@
 	9650 4000 9750 4000
 $Comp
-L power:GNDD #PWR061
+L power:GNDD #PWR068
 U 1 1 5EC6BDFB
 P 10050 4050
-F 0 "#PWR061" H 10050 3800 50  0001 C CNN
+F 0 "#PWR068" H 10050 3800 50  0001 C CNN
 F 1 "GNDD" H 10054 3895 50  0000 C CNN
 F 2 "" H 10050 4050 50  0001 C CNN
@@
 Text Notes 8350 4450 0    50   Italic 10
 Second microcontroller is added for possibility to use different package.\nSolder one microcontroller only.
-NoConn ~ 10450 3050
 NoConn ~ 10450 2850
 NoConn ~ 10450 2650
@@
 NoConn ~ 9150 2350
 NoConn ~ 9150 2050
-NoConn ~ 9150 1950
 Wire Wire Line
 	9650 950  9650 900
@@
 	10050 950  10050 900
 $Comp
-L MCU_ST_STM32F1:STM32F103CBUx U5
+L MCU_ST_STM32F1:STM32F103CBUx U6
 U 1 1 5EC6BE12
 P 9850 2450
-F 0 "U5" H 10150 900 50  0000 C CNN
+F 0 "U6" H 10150 900 50  0000 C CNN
 F 1 "STM32F103CBUx" H 10400 1000 50  0000 C CNN
 F 2 "Package_DFN_QFN:QFN-48-1EP_7x7mm_P0.5mm_EP5.6x5.6mm" H 9250 1050 50  0001 R CNN
@@
 Text GLabel 9150 1150 0    50   Input ~ 0
 SELF_NRST
-Text GLabel 9150 1850 0    50   Input ~ 0
-Board_ID
 Text GLabel 10450 2250 2    50   Input ~ 0
 AIN
@@
 	9950 900  10050 900
 $Comp
-L power:+3.3V #PWR056
+L power:+3.3V #PWR063
 U 1 1 5EC6FD9F
 P 9850 900
-F 0 "#PWR056" H 9850 750 50  0001 C CNN
+F 0 "#PWR063" H 9850 750 50  0001 C CNN
 F 1 "+3.3V" H 9865 1073 50  0000 C CNN
 F 2 "" H 9850 900 50  0001 C CNN
@@
 Self_RX(h)
 $Comp
-L power:GNDD #PWR058
+L power:GNDD #PWR065
 U 1 1 5F1BD152
 P 1250 2750
-F 0 "#PWR058" H 1250 2500 50  0001 C CNN
+F 0 "#PWR065" H 1250 2500 50  0001 C CNN
 F 1 "GNDD" H 1254 2595 50  0000 C CNN
 F 2 "" H 1250 2750 50  0001 C CNN
@@
 Self_SWDIO(h)
 $Comp
-L power:+3V3 #PWR057
+L power:+3V3 #PWR064
 U 1 1 5F1BD15D
 P 1250 1350
-F 0 "#PWR057" H 1250 1200 50  0001 C CNN
+F 0 "#PWR064" H 1250 1200 50  0001 C CNN
 F 1 "+3V3" H 1265 1523 50  0000 C CNN
 F 2 "" H 1250 1350 50  0001 C CNN
@@
 NoConn ~ 1750 2050
 $Comp
-L Connector:Conn_ST_STDC14 J6
+L Connector:Conn_ST_STDC14 J5
 U 1 1 5F1BD164
 P 1250 2050
-F 0 "J6" H 807 2096 50  0000 R CNN
+F 0 "J5" H 807 2096 50  0000 R CNN
 F 1 "Self" H 807 2005 50  0000 R CNN
 F 2 "Connector_PinHeader_1.27mm:PinHeader_2x07_P1.27mm_Vertical_SMD" H 1250 2050 50  0001 C CNN
@@
 NoConn ~ 1150 2750
 $Comp
-L Connector_Generic:Conn_01x04 J7
+L Connector_Generic:Conn_01x04 J6
 U 1 1 600768A8
 P 4150 2300
-F 0 "J7" H 4230 2292 50  0000 L CNN
+F 0 "J6" H 4230 2292 50  0000 L CNN
 F 1 "Conn_01x04" H 4230 2201 50  0000 L CNN
 F 2 "Connector_PinSocket_2.54mm:PinSocket_1x04_P2.54mm_Vertical" H 4150 2300 50  0001 C CNN
@@
 $EndComp
 $Comp
-L Connector_Generic:Conn_01x04 J8
+L Connector_Generic:Conn_01x04 J7
 U 1 1 600773E2
 P 4150 2900
-F 0 "J8" H 4230 2892 50  0000 L CNN
+F 0 "J7" H 4230 2892 50  0000 L CNN
 F 1 "Conn_01x04" H 4230 2801 50  0000 L CNN
 F 2 "Connector_PinSocket_2.54mm:PinSocket_1x04_P2.54mm_Vertical" H 4150 2900 50  0001 C CNN
@@
 Self_TX(h)
 $Comp
-L power:+3V3 #PWR059
+L power:+3V3 #PWR066
 U 1 1 60078E2D
 P 3950 2800
-F 0 "#PWR059" H 3950 2650 50  0001 C CNN
+F 0 "#PWR066" H 3950 2650 50  0001 C CNN
 F 1 "+3V3" H 3965 2973 50  0000 C CNN
 F 2 "" H 3950 2800 50  0001 C CNN
@@
 $EndComp
 $Comp
-L power:GNDD #PWR060
+L power:GNDD #PWR067
 U 1 1 60079A8D
 P 3950 3100
-F 0 "#PWR060" H 3950 2850 50  0001 C CNN
+F 0 "#PWR067" H 3950 2850 50  0001 C CNN
 F 1 "GNDD" H 3954 2945 50  0000 C CNN
 F 2 "" H 3950 3100 50  0001 C CNN
@@
 	1    0    0    -1
 $EndComp
+Text GLabel 9150 1850 0    50   Input ~ 0
+Board_ID1
+Text GLabel 9150 1950 0    50   Input ~ 0
+Board_ID2
+Text GLabel 10450 3050 2    50   BiDi ~ 0
+MCO
 $EndSCHEMATC
