File: project files/protected/stlink.kicad_pcb (KiCad board)
At the start: 2 copper layers, 43.2 x 17.8 mm, 58 parts, among them J1 USB Type C, J2 STDC-14, J3 SWD, J4 SWIM+VCP, J5 Power Target, J6 Self, J7 Conn_01x04, J8 Conn_01x04, Q1 MMBT9013, U1 AMS1117-3.3, U2 USBLC6-2P6, U3 TXS0108EPW, U4 STM32F103CBTx, U5 STM32F103CBUx, Y1 8MHz

Commit message: Fixes
Parts:
- removed the J5 at (271.1, 127.0)
- removed the JP2 at (209.6, 124.5)
- removed the R11 at (259.7, 86.6)
- removed the R16 at (255.2, 91.6)
- removed the R9 at (255.7, 89.1)
- added C10: 100nF, Capacitor_SMD:C_0603_1608Metric, F.Cu at (235.7, 84.4)
- added C9: 100nF, Capacitor_SMD:C_0603_1608Metric, F.Cu at (241.3, 77.5)
- added R12: 100R, Resistor_SMD:R_0603_1608Metric, F.Cu at (241.3, 80.0)
- added R14: 100K, Resistor_SMD:R_0603_1608Metric, F.Cu at (245.3, 77.5)
- added R15: 100K, Resistor_SMD:R_0603_1608Metric, F.Cu at (239.7, 84.4)
- added R17: 10K, Resistor_SMD:R_0603_1608Metric, F.Cu at (245.3, 80.0)
- added R26: 100K, Resistor_SMD:R_0603_1608Metric, F.Cu at (174.0, 116.8)
- added SW1: Power Ext, Button_Switch_SMD:SW_SPDT_PCM12, F.Cu at (232.4, 123.8)
- added U4: 74LVC2G07, Package_TO_SOT_SMD:SOT-363_SC-70-6, F.Cu at (231.6, 85.0)
- R25: renamed from R24; value 10K -> 100K
- renumbered C9 to C11, C10 to C12, C11 to C13, C12 to C14, C13 to C15, J6 to J5, J7 to J6, J8 to J7, JP1 to JP2, R12 to R10, R13 to R11, R15 to R13, R14 to R16, R17 to R18, R18 to R20, R20 to R21, R21 to R22, R22 to R23, R23 to R24, R10 to R9, U4 to U5, U5 to U6
Connections:
- net Board_ID renamed Board_ID1
- net Net-(D1-Pad2) renamed +5V
- C1 pad 2: GNDD -> GND
- C11 pad 1: GNDD -> GND
- C12 pad 1: GNDD -> GND
- C12 pad 2: SELF_NRST -> Self_NRST
- C13 pad 1: GNDD -> GND
- C14 pad 2: GNDD -> GND
- C15 pad 2: GNDD -> GND
- C2 pad 2: GNDD -> GND
- C3 pad 2: GNDD -> GND
- C4 pad 2: GNDD -> GND
- C5 pad 2: GNDD -> GND
- C6 pad 2: GNDD -> GND
- C7 pad 2: GNDD -> GND
- C8 pad 2: GNDD -> GND
- D3 pad 1: GNDD -> GND
- J1 pad A1: GNDD -> GND
- J1 pad A12: GNDD -> GND
- J1 pad A6: Net-(J1-PadA6) -> /D+
- J1 pad A7: Net-(J1-PadA7) -> /D-
- J1 pad B1: GNDD -> GND
- J1 pad B12: GNDD -> GND
- J1 pad B6: Net-(J1-PadA6) -> /D+
- J1 pad B7: Net-(J1-PadA7) -> /D-
- J1 pad S1: Net-(J1-PadS1) -> GND
- J2 pad 11: GNDD -> GND
- J2 pad 5: GNDD -> GND
- J2 pad 7: GNDD -> GND
- J3 pad 3: GNDD -> GND
- J4 pad 3: GNDD -> GND
- J5 pad 12: SELF_NRST -> Self_NRST
- J5 pad 4: SWDIO -> Self_SWDIO
- J5 pad 5: GNDD -> GND
- J5 pad 6: SWDCLK -> Self_SWDCLK
- J5 pad 7: GNDD -> GND
- J5 pad 8: SWO -> Self_SWO
- J6 pad 1: SELF_NRST -> Self_NRST
- J6 pad 2: SWDCLK -> Self_SWDCLK
- J6 pad 3: SWDIO -> Self_SWDIO
- J6 pad 4: SWO -> Self_SWO
- J7 pad 4: GNDD -> GND
- R13 pad 1: GNDD -> GND
- R16 pad 1: GNDD -> GND
- R2 pad 2: GNDD -> GND
- R22 pad 2: GNDD -> GND
- R23 pad 2: GNDD -> GND
- R24 pad 2: SELF_NRST -> Self_NRST
- R25 pad 2: GNDD -> GND
- R3 pad 2: GNDD -> GND
- R6 pad 2: GNDD -> GND
- R7 pad 1: GNDD -> GND
- U1 pad 1: GNDD -> GND
- U2 pad 2: GNDD -> GND
- U3 pad 11: GNDD -> GND
- U3 pad 13: T_NRST_SWIM -> T_JTDI
- U3 pad 17: T_NRST_SWD -> Net-(U3-Pad17)
- U3 pad 20: SWDCLK -> T_SWDCLK
- U3 pad 4: T_NRST_SWD(h) -> Net-(U3-Pad4)
- U3 pad 8: T_NRST_SWIM(h) -> T_JTDI(h)
- U5 pad 20: GNDD -> BOOT_1
- U5 pad 23: GNDD -> GND
- U5 pad 29: Net-(U4-Pad29) -> MCO
- U5 pad 3: Net-(U4-Pad3) -> Board_ID2
- U5 pad 34: SWDIO -> Self_SWDIO
- U5 pad 35: GNDD -> GND
- U5 pad 37: SWDCLK -> Self_SWDCLK
- U5 pad 39: SWO -> Self_SWO
- U5 pad 47: GNDD -> GND
- U5 pad 7: SELF_NRST -> Self_NRST
- U5 pad 8: GNDD -> GND
- U6 pad 23: GNDD -> GND
- U6 pad 29: Net-(U5-Pad29) -> MCO
- U6 pad 3: Net-(U5-Pad3) -> Board_ID2
- U6 pad 35: GNDD -> GND
- U6 pad 47: GNDD -> GND
- U6 pad 49: GNDD -> GND
- U6 pad 8: GNDD -> GND
- Y1 pad 2: GNDD -> GND
- Y1 pad 4: GNDD -> GND
