File: project files/protected/stlink.sch (KiCad schematic (older format))
At the start: 53 parts, among them J1 USB Type C, J2 STDC-14, J3 SWD, J4 SWIM+VCP, J5 Power Target, Q1 MMBT9013, U1 AMS1117-3.3, U2 USBLC6-2P6, U3 TXS0108EPW, U4 STM32F103CBTx, Y1 8MHz

Commit message: Fixes
Parts:
- removed J5: Power Target, Connector_PinHeader_2.54mm:PinHeader_2x02_P2.54mm_Vertical, symbol Connector_Generic:Conn_02x02_Odd_Even
- removed R11, R9: 22R, Resistor_SMD:R_0603_1608Metric, symbol Device:R
- removed R16: 47R, Resistor_SMD:R_0603_1608Metric, symbol Device:R
- added C10, C9: 100nF, Capacitor_SMD:C_0603_1608Metric, symbol Device:C
- added R12: 100R, Resistor_SMD:R_0603_1608Metric, symbol Device:R
- added R14, R15, R26: 100K, Resistor_SMD:R_0603_1608Metric, symbol Device:R
- added R17: 10K, Resistor_SMD:R_0603_1608Metric, symbol Device:R
- added SW1: Power Ext, Button_Switch_SMD:SW_SPDT_PCM12, symbol Switch:SW_Push_SPDT
- added U4: 74LVC2G07, Package_TO_SOT_SMD:SOT-363_SC-70-6, symbol 74xGxx:74LVC2G07
- R25: renamed from R24; value 10K -> 100K
- renumbered C9 to C11, C10 to C12, C11 to C13, C12 to C14, C13 to C15, JP1 to JP2, R12 to R10, R13 to R11, R15 to R13, R14 to R16, R17 to R18, R18 to R20, R20 to R21, R21 to R22, R22 to R23, R23 to R24, R10 to R9, U4 to U5
Connections:
- net +3V3: now also C10.2, R14.1, R15.1, SW1.1 (A), U4.5 (VCC), U4.5 (VCC)
- net D+: now also J1.A6 (D+), J1.B6 (D+)
- net D-: now also J1.A7 (D-), J1.B7 (D-)
- net T_JTDI: now also U3.13 (B7)
- net T_JTDI(h): now also U3.8 (A7)
- net T_NRST_SWD: now also R14.2, U4.1; no longer U3.17 (B3)
- net T_NRST_SWD(h): now also U4.6; no longer U3.4 (A3)
- net T_NRST_SWIM: now also R15.2, U4.3; no longer U3.13 (B7)
- net T_NRST_SWIM(h): now also U4.4; no longer U3.8 (A7)
- net T_SWDCLK: now also U3.20 (B1)
- net T_Vref: now also SW1.2 (B)
- net VBUS: now also C9.1
- net +5V: now reaches D1.2 (A), J1.A4 (VBUS), J1.A9 (VBUS), J1.B4 (VBUS), J1.B9 (VBUS)
- net GND: now reaches J1.S1 (SHIELD)
- net GND: now also C1.2, C11.1, C12.1, C13.1, C14.2, C15.2, C2.2, C3.2, C4.2, C5.2, C6.2, C7.2, C8.2, D3.1 (A1), J1.A1 (GND), J1.A12 (GND), J1.B1 (GND), J1.B12 (GND), J2.11 (GNDDetect), J2.5 (GND), J2.7 (GND), J3.3 (Pin_3), J4.3 (Pin_3), R13.1, R16.1, R2.2, R22.2, R23.2, R25.2, R3.2, R6.2, R7.1, U1.1 (GND), U2.2 (GND), U3.11 (GND), U5.23 (VSS), U5.35 (VSS), U5.47 (VSS), U5.8 (VSSA), Y1.2, Y1.4, C10.1, C9.2, R17.1, R26.2, U4.2 (GND), U4.2 (GND)
- net MCO: now reaches U5.29 (PA8)
- net MCO: now also R12.2
- net Board_ID2: now reaches U5.3 (PC14)
- net Board_ID2: now also R17.2
- net Board_ID renamed Board_ID1
- removed net GNDD: C1.2, C11.1, C12.1, C13.1, C14.2, C15.2, C2.2, C3.2, C4.2, C5.2, C6.2, C7.2, C8.2, D3.1 (A1), J1.A1 (GND), J1.A12 (GND), J1.B1 (GND), J1.B12 (GND), J2.11 (GNDDetect), J2.5 (GND), J2.7 (GND), J3.3 (Pin_3), J4.3 (Pin_3), R13.1, R16.1, R2.2, R22.2, R23.2, R25.2, R3.2, R6.2, R7.1, U1.1 (GND), U2.2 (GND), U3.11 (GND), U5.20 (PB2), U5.23 (VSS), U5.35 (VSS), U5.47 (VSS), U5.8 (VSSA), Y1.2, Y1.4
- net SELF_NRST renamed Self_NRST
- net SWDCLK renamed Self_SWDCLK
- net Self_SWDCLK: no longer U3.20 (B1)
- net SWDIO renamed Self_SWDIO
- net SWO renamed Self_SWO
- new net BOOT_1: R26.1, U5.20 (PB2)
- new net T_MCO: R12.1
Other:
- note added: "Decoupling capacitors:\none per each VDD, VDA, VBAT of MCU\nand USBLC6-2P6"
- note added: "Don't fit Board_ID2\nresistor"
- note added: "Jumper for powering target from ST-Link"
- note added: "STLINK_USB_D(+) and STLINK_USB_D(-):\nshould be a differential pair approx. 90 Ohm\nLength diference of those traces must be <1.1 mm"
- note added: "or MMBT2222A"
- note removed: "Decoupling capacitors:\none per each VDD, VDA, and VBAT"
- note removed: "STLINK_USB_D(+) and STLINK_USB_D(-):\nshould be a differential pair approx. 90 Ohm\nLength diference of those traces \nmust be <1.1 mm\nthe 22 Ohm resistros can be replaced by 0 Ohms."
- note removed: "Vref PullDown\ncan be 10K"
- moved on the sheet: C11, C12, C13, C14, D1, D3, D4, JP2, R16, R18, R19, R20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
